File: bms_master_pcb2/bms_master_pcb2.kicad_sch (KiCad schematic)
At the start: 22 parts, among them J101 EXTRA COMMS, J102 GPIO, J103 EXTRA POWER, J104 TC2030, J105 EXTRA BMS OUTPUTS, J106 OUT, U101 STM32G474RETx, U102 SST26VF064B-104V/MF

Commit message: Add files via upload
almost done with the PCB layout. Harrison needs to fix routing on the differential pairs
Parts:
- added H101, H102, H103, H104: MountingHole, MountingHole:MountingHole_3.2mm_M3_Pad, symbol Mechanical:MountingHole_Pad
- C101, C106, C110: footprint (none) -> Capacitor_SMD:C_0805_2012Metric_Pad1.18x1.45mm_HandSolder
- C102, C103, C104, C105, C107, C108, C109: footprint (none) -> Capacitor_SMD:C_0603_1608Metric_Pad1.08x0.95mm_HandSolder
- J101, J102, J106: footprint (none) -> Connector_PinHeader_2.54mm:PinHeader_1x10_P2.54mm_Vertical
- J103: footprint (none) -> Connector_PinHeader_2.54mm:PinHeader_1x04_P2.54mm_Vertical
- J105: footprint (none) -> Connector_PinHeader_2.54mm:PinHeader_1x05_P2.54mm_Vertical
- L101, L102: footprint (none) -> bms_master_pcb2:WE-HEPC_6030
- R101, R102: footprint (none) -> Resistor_SMD:R_0603_1608Metric_Pad0.98x0.95mm_HandSolder
- U102: footprint (none) -> Package_DFN_QFN:WDFN-8-1EP_6x5mm_P1.27mm_EP3.4x4mm
Connections:
- net GND: now also H101.1, H102.1, H103.1, H104.1

Commit message: Add files via upload
finished and ready to order V1.01
Parts:
- removed J105: EXTRA BMS OUTPUTS, Connector_PinHeader_2.54mm:PinHeader_1x05_P2.54mm_Vertical, symbol Connector:Conn_01x05_Pin
- removed J106: OUT, Connector_PinHeader_2.54mm:PinHeader_1x10_P2.54mm_Vertical, symbol Connector:Conn_01x10_Pin
- added J105: EXTRA BMS OUTPUTS, Connector_PinHeader_2.54mm:PinHeader_1x07_P2.54mm_Vertical, symbol Connector:Conn_01x07_Pin
- added J106: OUT, Connector_PinHeader_2.54mm:PinHeader_1x06_P2.54mm_Vertical, symbol Connector:Conn_01x06_Pin
Connections:
- net CLK is gone; now on net QSPI.CLK: U102.6 (SCK)
- net IO0 is gone; now on net QSPI.IO0: U102.5 (SI)
- net IO1 is gone; now on net QSPI.IO1: U102.2 (SO)
- net IO2 is gone; now on net QSPI.IO2: U102.3 (WP#)
- net IO3 is gone; now on net QSPI.IO3: U102.7 (HOLD)
- net NCS is gone; now on net QSPI.NCS: U102.1 (CE#)
- net +12V: now also J106.1 (Pin_1)
- net Digital Outputs and Happy Lights/BMS_OUT_0: now also J105.1 (Pin_1)
- net Digital Outputs and Happy Lights/BMS_OUT_1: now also J105.2 (Pin_2)
- net Digital Outputs and Happy Lights/BMS_OUT_2: now also J105.3 (Pin_3)
- net Digital Outputs and Happy Lights/BMS_OUT_3: now also J105.4 (Pin_4)
- net Digital Outputs and Happy Lights/BMS_OUT_4: now also J105.5 (Pin_5)
- net Digital Outputs and Happy Lights/BMS_OUT_5: now also J105.6 (Pin_6)
- net Digital Outputs and Happy Lights/BMS_OUT_6: now also J105.7 (Pin_7)
- net GND: now also J106.6 (Pin_6)
- net FDCAN3_RX renamed FDCAN3.D-
- net FDCAN3_TX renamed FDCAN3.D+
- new net CAN.1+: J106.3 (Pin_3)
- new net CAN.1-: J106.2 (Pin_2)
- new net CAN.2+: J106.4 (Pin_4)
- new net CAN.2-: J106.5 (Pin_5)
- no-connect marks 8 -> 10
Other:
- sheet CAN ports: added CAN{1+ 1-}, CAN{2+ 2-}; removed CAN1{H L}, CAN2{H L}
- note added: "H"
- note added: "L"
- note added: "RX"
- note added: "TX"
