File: bms_master_pcb2/can.kicad_sch (KiCad schematic)
At the start: 12 parts, among them U401 TCAN1044AVDDFRQ1, U402 TCAN1044AVDDFRQ1

Commit message: Add files via upload
almost done with the PCB layout. Harrison needs to fix routing on the differential pairs
Parts:
- C401, C402, C403, C404, C405, C406: footprint (none) -> Capacitor_SMD:C_0603_1608Metric_Pad1.08x0.95mm_HandSolder
- R401, R402, R403, R404: footprint (none) -> Resistor_SMD:R_1206_3216Metric_Pad1.30x1.75mm_HandSolder
- U401, U402: footprint (none) -> Package_TO_SOT_SMD:TSOT-23-8_HandSoldering
Other:
- note added: "could only find 1206 size 60ohm Resistors"
- note added: "output characteristic impediance 120 ohms"
Changed lines of the file:
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@@
 	(generator_version "10.0")
 	(paper "A4")
+	(text "output characteristic impediance 120 ohms"
+		(exclude_from_sim no)
+		(at 211.328 82.296 0)
+		(effects
+			(font
+				(size 1.27 1.27)
+			)
+		)
+	)
+	(text "could only find 1206 size 60ohm Resistors"
+		(exclude_from_sim no)
+		(at 197.104 43.942 0)
+		(effects
+			(font
+				(size 1.27 1.27)
+			)
+		)
+	)
 	(junction
 		(at 195.58 55.88)
@@
 			)
 		)
-		(property "Footprint" ""
+		(property "Footprint" "Capacitor_SMD:C_0603_1608Metric_Pad1.08x0.95mm_HandSolder"
 			(at 101.6 82.55 0)
 			(hide yes)
@@
 			)
 		)
-		(property "Footprint" ""
+		(property "Footprint" "Package_TO_SOT_SMD:TSOT-23-8_HandSoldering"
 			(at 156.21 45.72 0)
 			(hide yes)
@@
 			)
 		)
-		(property "Footprint" ""
+		(property "Footprint" "Resistor_SMD:R_1206_3216Metric_Pad1.30x1.75mm_HandSolder"
 			(at 195.58 95.25 0)
 			(hide yes)
@@
 			)
 		)
-		(property "Footprint" ""
+		(property "Footprint" "Capacitor_SMD:C_0603_1608Metric_Pad1.08x0.95mm_HandSolder"
 			(at 101.6 44.45 0)
 			(hide yes)
@@
 			)
 		)
-		(property "Footprint" ""
+		(property "Footprint" "Capacitor_SMD:C_0603_1608Metric_Pad1.08x0.95mm_HandSolder"
 			(at 113.03 82.55 0)
 			(hide yes)
@@
 			)
 		)
-		(property "Footprint" ""
+		(property "Footprint" "Resistor_SMD:R_1206_3216Metric_Pad1.30x1.75mm_HandSolder"
 			(at 195.58 105.41 0)
 			(hide yes)
@@
 			)
 		)
-		(property "Footprint" ""
+		(property "Footprint" "Capacitor_SMD:C_0603_1608Metric_Pad1.08x0.95mm_HandSolder"
 			(at 113.03 44.45 0)
 			(hide yes)
@@
 			)
 		)
-		(property "Footprint" ""
+		(property "Footprint" "Resistor_SMD:R_1206_3216Metric_Pad1.30x1.75mm_HandSolder"
 			(at 195.58 68.58 0)
 			(hide yes)
@@
 			)
 		)
-		(property "Footprint" ""
+		(property "Footprint" "Package_TO_SOT_SMD:TSOT-23-8_HandSoldering"
 			(at 156.21 82.55 0)
 			(hide yes)
@@
 			)
 		)
-		(property "Footprint" ""
+		(property "Footprint" "Capacitor_SMD:C_0603_1608Metric_Pad1.08x0.95mm_HandSolder"
 			(at 200.66 63.5 0)
 			(hide yes)
@@
 			)
 		)
-		(property "Footprint" ""
+		(property "Footprint" "Capacitor_SMD:C_0603_1608Metric_Pad1.08x0.95mm_HandSolder"
 			(at 200.66 100.33 0)
 			(hide yes)
@@
 			)
 		)
-		(property "Footprint" ""
+		(property "Footprint" "Resistor_SMD:R_1206_3216Metric_Pad1.30x1.75mm_HandSolder"
 			(at 195.58 58.42 0)
 			(hide yes)

Commit message: Add files via upload
finished and ready to order V1.01
Connections:
- net CAN1.H renamed CAN.1+
- net CAN1.L renamed CAN.1-
- net CAN2.H renamed CAN.2+
- net CAN2.L renamed CAN.2-
Other:
- note added: "H"
- note added: "L"
Changed lines of the file:
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@@
 	(generator_version "10.0")
 	(paper "A4")
+	(text "L"
+		(exclude_from_sim no)
+		(at 171.958 100.33 0)
+		(effects
+			(font
+				(size 1.27 1.27)
+			)
+		)
+	)
+	(text "H"
+		(exclude_from_sim no)
+		(at 171.704 98.044 0)
+		(effects
+			(font
+				(size 1.27 1.27)
+			)
+		)
+	)
 	(text "output characteristic impediance 120 ohms"
 		(exclude_from_sim no)
@@
 		)
 	)
+	(text "L"
+		(exclude_from_sim no)
+		(at 171.958 63.5 0)
+		(effects
+			(font
+				(size 1.27 1.27)
+			)
+		)
+	)
 	(text "could only find 1206 size 60ohm Resistors"
 		(exclude_from_sim no)
 		(at 197.104 43.942 0)
+		(effects
+			(font
+				(size 1.27 1.27)
+			)
+		)
+	)
+	(text "H"
+		(exclude_from_sim no)
+		(at 171.704 61.214 0)
 		(effects
 			(font
@@
 		)
 	)
-	(label "CAN2.H"
-		(at 171.45 99.06 0)
-		(effects
-			(font
-				(size 1.27 1.27)
-			)
-			(justify left bottom)
-		)
-	)
 	(label "CAN1.RX"
 		(at 129.54 64.77 0)
@@
 		)
 	)
-	(label "CAN2.L"
-		(at 171.45 101.6 0)
+	(label "CAN.2-"
+		(at 173.99 101.6 0)
+		(effects
+			(font
+				(size 1.27 1.27)
+			)
+			(justify left bottom)
+		)
+	)
+	(label "CAN.1-"
+		(at 173.99 64.77 0)
+		(effects
+			(font
+				(size 1.27 1.27)
+			)
+			(justify left bottom)
+		)
+	)
+	(label "CAN.1+"
+		(at 173.99 62.23 0)
 		(effects
 			(font
@@
 		)
 	)
-	(label "CAN1.H"
-		(at 171.45 62.23 0)
-		(effects
-			(font
-				(size 1.27 1.27)
-			)
-			(justify left bottom)
-		)
-	)
 	(label "CAN2.TX"
 		(at 129.54 99.06 0)
@@
 		)
 	)
-	(label "CAN1.L"
-		(at 171.45 64.77 0)
-		(effects
-			(font
-				(size 1.27 1.27)
-			)
-			(justify left bottom)
-		)
-	)
 	(label "CAN1.TX"
 		(at 129.54 62.23 0)
+		(effects
+			(font
+				(size 1.27 1.27)
+			)
+			(justify left bottom)
+		)
+	)
+	(label "CAN.2+"
+		(at 173.99 99.06 0)
 		(effects
 			(font
@@
 		)
 	)
-	(hierarchical_label "CAN2{H L}"
+	(hierarchical_label "CAN{2+ 2-}"
 		(shape input)
 		(at 231.14 96.52 0)
@@
 		)
 	)
-	(hierarchical_label "CAN1{H L}"
+	(hierarchical_label "CAN{1+ 1-}"
 		(shape input)
 		(at 231.14 59.69 0)
