File: bms_master_pcb2/isospi.kicad_sch (KiCad schematic)
At the start: 19 parts, among them J201 Conn_01x04, J202 Conn_01x04, U201 LTC6820HMS-TRPBF, U202 LTC6820HMS-TRPBF

Commit message: Add files via upload
almost done with the PCB layout. Harrison needs to fix routing on the differential pairs
Parts:
- C201, C202: footprint (none) -> Capacitor_SMD:C_0603_1608Metric_Pad1.08x0.95mm_HandSolder
- J201, J202: footprint (none) -> Connector_Molex:Molex_Micro-Fit_3.0_43650-0400_1x04_P3.00mm_Horizontal
- R201, R203, R204, R205, R206, R207, R208, R209, R210, R211, R212: footprint (none) -> Resistor_SMD:R_0603_1608Metric_Pad0.98x0.95mm_HandSolder
- R202: footprint (none) -> Resistor_SMD:R_0603_1608Metric_Pad0.98x0.95mm_HandSolder; now not fitted
- U201, U202: footprint MS_05-08-1669_ADI -> bms_master_pcb2:MS_05-08-1669_ADI
Connections:
- net E-METER_PASSTHROUGH_1: now also J201.1 (Pin_1), J202.1 (Pin_1); no longer J201.3 (Pin_3), J202.3 (Pin_3)
- net E-METER_PASSTHROUGH_2: now also J201.2 (Pin_2), J202.2 (Pin_2); no longer J201.4 (Pin_4), J202.4 (Pin_4)
- net at TR201.1 (TX-): now also J202.3 (Pin_3); no longer J201.1 (Pin_1)
- net at TR201.3 (TX+): now also J202.4 (Pin_4); no longer J201.2 (Pin_2)
- net at TR201.6 (RX-): now also J201.3 (Pin_3); no longer J202.1 (Pin_1)
- net at TR201.8 (RX+): now also J201.4 (Pin_4); no longer J202.2 (Pin_2)
Other:
- note added: "2 pull-ups?"
- moved on the sheet: J201, J202
Changed lines of the file:
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@@
 	(generator_version "10.0")
 	(paper "A4")
+	(text "2 pull-ups?"
+		(exclude_from_sim no)
+		(at 37.084 76.454 0)
+		(effects
+			(font
+				(size 1.27 1.27)
+			)
+		)
+	)
 	(junction
 		(at 104.14 38.1)
@@
 	(hierarchical_label "E-METER_PASSTHROUGH_1"
 		(shape input)
-		(at 218.44 87.63 180)
+		(at 218.44 77.47 180)
 		(effects
 			(font
@@
 	(hierarchical_label "E-METER_PASSTHROUGH_1"
 		(shape input)
-		(at 218.44 74.93 180)
+		(at 218.44 64.77 180)
 		(effects
 			(font
@@
 	(hierarchical_label "E-METER_PASSTHROUGH_2"
 		(shape input)
-		(at 218.44 77.47 180)
+		(at 218.44 67.31 180)
 		(effects
 			(font
@@
 	(hierarchical_label "E-METER_PASSTHROUGH_2"
 		(shape input)
-		(at 218.44 90.17 180)
+		(at 218.44 80.01 180)
 		(effects
 			(font
@@
 			)
 		)
-		(property "Footprint" ""
+		(property "Footprint" "Resistor_SMD:R_0603_1608Metric_Pad0.98x0.95mm_HandSolder"
 			(at 90.17 88.9 0)
 			(hide yes)
@@
 			)
 		)
-		(property "Footprint" ""
+		(property "Footprint" "Capacitor_SMD:C_0603_1608Metric_Pad1.08x0.95mm_HandSolder"
 			(at 146.05 82.55 0)
 			(hide yes)
@@
 			)
 		)
-		(property "Footprint" ""
+		(property "Footprint" "Resistor_SMD:R_0603_1608Metric_Pad0.98x0.95mm_HandSolder"
 			(at 88.9 46.99 0)
 			(hide yes)
@@
 			)
 		)
-		(property "Footprint" ""
+		(property "Footprint" "Resistor_SMD:R_0603_1608Metric_Pad0.98x0.95mm_HandSolder"
 			(at 80.01 27.94 0)
 			(hide yes)
@@
 			)
 		)
-		(property "Footprint" ""
+		(property "Footprint" "Resistor_SMD:R_0603_1608Metric_Pad0.98x0.95mm_HandSolder"
 			(at 109.22 38.1 0)
 			(hide yes)
@@
 			)
 		)
-		(property "Footprint" "MS_05-08-1669_ADI"
+		(property "Footprint" "bms_master_pcb2:MS_05-08-1669_ADI"
 			(at 72.39 76.454 0)
 			(hide yes)
@@
 			)
 		)
-		(property "Footprint" ""
+		(property "Footprint" "Resistor_SMD:R_0603_1608Metric_Pad0.98x0.95mm_HandSolder"
 			(at 109.22 88.9 0)
 			(hide yes)
@@
 	(symbol
 		(lib_id "Connector_Generic:Conn_01x04")
-		(at 223.52 72.39 0)
+		(at 223.52 80.01 0)
 		(unit 1)
 		(body_style 1)
@@
 		(fields_autoplaced yes)
 		(property "Reference" "J201"
-			(at 226.06 72.3899 0)
+			(at 226.06 80.0099 0)
 			(show_name no)
 			(do_not_autoplace no)
@@
 		)
 		(property "Value" "Conn_01x04"
-			(at 226.06 74.9299 0)
+			(at 226.06 82.5499 0)
 			(show_name no)
 			(do_not_autoplace no)
@@
 			)
 		)
-		(property "Footprint" ""
-			(at 223.52 72.39 0)
+		(property "Footprint" "Connector_Molex:Molex_Micro-Fit_3.0_43650-0400_1x04_P3.00mm_Horizontal"
+			(at 223.52 80.01 0)
 			(hide yes)
 			(show_name no)
@@
 		)
 		(property "Datasheet" ""
-			(at 223.52 72.39 0)
+			(at 223.52 80.01 0)
 			(hide yes)
 			(show_name no)
@@
 		)
 		(property "Description" "Generic connector, single row, 01x04, script generated (kicad-library-utils/schlib/autogen/connector/)"
-			(at 223.52 72.39 0)
+			(at 223.52 80.01 0)
 			(hide yes)
 			(show_name no)
@@
 			)
 		)
-		(property "Footprint" ""
+		(property "Footprint" "Resistor_SMD:R_0603_1608Metric_Pad0.98x0.95mm_HandSolder"
 			(at 88.9 100.33 0)
 			(hide yes)
@@
 		(on_board yes)
 		(in_pos_files yes)
-		(dnp no)
+		(dnp yes)
 		(fields_autoplaced yes)
 		(property "Reference" "R202"
@@
 			)
 		)
-		(property "Footprint" ""
+		(property "Footprint" "Resistor_SMD:R_0603_1608Metric_Pad0.98x0.95mm_HandSolder"
 			(at 35.56 91.44 0)
 			(hide yes)
@@
 			)
 		)
-		(property "Footprint" ""
+		(property "Footprint" "Capacitor_SMD:C_0603_1608Metric_Pad1.08x0.95mm_HandSolder"
 			(at 146.05 72.39 0)
 			(hide yes)
@@
 			)
 		)
-		(property "Footprint" ""
+		(property "Footprint" "Resistor_SMD:R_0603_1608Metric_Pad0.98x0.95mm_HandSolder"
 			(at 35.56 38.1 0)
 			(hide yes)
@@
 			)
 		)
-		(property "Footprint" ""
+		(property "Footprint" "Resistor_SMD:R_0603_1608Metric_Pad0.98x0.95mm_HandSolder"
 			(at 109.22 91.44 0)
 			(hide yes)
@@
 	(symbol
 		(lib_id "Connector_Generic:Conn_01x04")
-		(at 223.52 85.09 0)
+		(at 223.52 67.31 0)
 		(unit 1)
 		(body_style 1)
@@
 		(fields_autoplaced yes)
 		(property "Reference" "J202"
-			(at 226.06 85.0899 0)
+			(at 226.06 67.3099 0)
 			(show_name no)
 			(do_not_autoplace no)
@@
 		)
 		(property "Value" "Conn_01x04"
-			(at 226.06 87.6299 0)
+			(at 226.06 69.8499 0)
 			(show_name no)
 			(do_not_autoplace no)
@@
 			)
 		)
-		(property "Footprint" ""
-			(at 223.52 85.09 0)
+		(property "Footprint" "Connector_Molex:Molex_Micro-Fit_3.0_43650-0400_1x04_P3.00mm_Horizontal"
+			(at 223.52 67.31 0)
 			(hide yes)
 			(show_name no)
@@
 		)
 		(property "Datasheet" ""
-			(at 223.52 85.09 0)
+			(at 223.52 67.31 0)
 			(hide yes)
 			(show_name no)
@@
 		)
 		(property "Description" "Generic connector, single row, 01x04, script generated (kicad-library-utils/schlib/autogen/connector/)"
-			(at 223.52 85.09 0)
+			(at 223.52 67.31 0)
 			(hide yes)
 			(show_name no)
@@
 			)
 		)
-		(property "Footprint" ""
+		(property "Footprint" "Resistor_SMD:R_0603_1608Metric_Pad0.98x0.95mm_HandSolder"
 			(at 90.17 35.56 0)
 			(hide yes)
@@
 			)
 		)
-		(property "Footprint" "MS_05-08-1669_ADI"
+		(property "Footprint" "bms_master_pcb2:MS_05-08-1669_ADI"
 			(at 72.39 23.114 0)
 			(hide yes)
@@
 			)
 		)
-		(property "Footprint" ""
+		(property "Footprint" "Resistor_SMD:R_0603_1608Metric_Pad0.98x0.95mm_HandSolder"
 			(at 109.22 35.56 0)
 			(hide yes)
@@
 			)
 		)
-		(property "Footprint" ""
+		(property "Footprint" "Resistor_SMD:R_0603_1608Metric_Pad0.98x0.95mm_HandSolder"
 			(at 80.01 81.28 0)
 			(hide yes)

Commit message: Add files via upload
finished and ready to order V1.01
Connections:
- net isoSPI.D-: now reaches R205.1, U201.10 (IM)
- net isoSPI.D-: now also TR201.16 (TD+); no longer TR201.14 (TD+)
- net isoSPI.D+: now reaches R205.2, U201.11 (IP)
- net isoSPI.D+: now also TR201.14 (TD-); no longer TR201.16 (TD-)
- net isoSPI_2.D-: now reaches R206.1, U202.10 (IM)
- net isoSPI_2.D-: now also TR201.11 (RD+); no longer TR201.9 (RD+)
- net isoSPI_2.D+: now reaches R206.2, U202.11 (IP)
- net isoSPI_2.D+: now also TR201.9 (RD-); no longer TR201.11 (RD-)
- net INPUT_isoSPI.D+: now reaches J202.3 (Pin_3)
- net INPUT_isoSPI.D+: now also TR201.3 (TX-); no longer TR201.1 (TX-)
- net INPUT_isoSPI.D-: now reaches J202.4 (Pin_4)
- net INPUT_isoSPI.D-: now also TR201.1; no longer TR201.3 (TX+)
- net OUTPUT_isoSPI.D+: now reaches J201.3 (Pin_3)
- net OUTPUT_isoSPI.D+: now also TR201.8 (RX-); no longer TR201.6 (RX-)
- net OUTPUT_isoSPI.D-: now reaches J201.4 (Pin_4)
- net OUTPUT_isoSPI.D-: now also TR201.6 (RX+); no longer TR201.8 (RX+)
Changed lines of the file:
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@@
+		)
+	)
+	(label "isoSPI.D+"
+		(at 129.54 44.45 0)
+		(effects
+			(font
+				(size 1.27 1.27)
+			)
+			(justify left bottom)
 		)
 	)
@@
 		)
 	)
+	(label "isoSPI_2.D+"
+		(at 118.11 97.79 0)
+		(effects
+			(font
+				(size 1.27 1.27)
+			)
+			(justify left bottom)
+		)
+	)
+	(label "OUTPUT_isoSPI.D+"
+		(at 182.88 82.55 0)
+		(effects
+			(font
+				(size 1.27 1.27)
+			)
+			(justify left bottom)
+		)
+	)
+	(label "INPUT_isoSPI.D-"
+		(at 181.61 72.39 0)
+		(effects
+			(font
+				(size 1.27 1.27)
+			)
+			(justify left bottom)
+		)
+	)
 	(label "SPI2.SCK"
 		(at 46.99 96.52 0)
@@
 		)
 	)
+	(label "INPUT_isoSPI.D+"
+		(at 181.61 69.85 0)
+		(effects
+			(font
+				(size 1.27 1.27)
+			)
+			(justify left bottom)
+		)
+	)
 	(label "SPI2.MISO"
 		(at 46.99 40.64 0)
@@
 		)
 	)
+	(label "OUTPUT_isoSPI.D-"
+		(at 182.88 85.09 0)
+		(effects
+			(font
+				(size 1.27 1.27)
+			)
+			(justify left bottom)
+		)
+	)
+	(label "isoSPI.D-"
+		(at 124.46 49.53 0)
+		(effects
+			(font
+				(size 1.27 1.27)
+			)
+			(justify left bottom)
+		)
+	)
 	(label "SPI2.MOSI"
 		(at 46.99 38.1 0)
@@
 	(label "SPI2.MISO"
 		(at 46.99 93.98 0)
+		(effects
+			(font
+				(size 1.27 1.27)
+			)
+			(justify left bottom)
+		)
+	)
+	(label "isoSPI_2.D-"
+		(at 118.11 102.87 0)
 		(effects
 			(font
@@
 			)
 		)
+		(pin "1"
+		)
+		(pin "7"
+		)
+		(pin "5"
+		)
+		(pin "8"
+		)
+		(pin "12"
+		)
+		(pin "11"
+		)
 		(pin "3"
 		)
-		(pin "7"
-		)
-		(pin "5"
-		)
-		(pin "8"
-		)
-		(pin "12"
-		)
-		(pin "11"
-		)
-		(pin "1"
-		)
 		(pin "6"
