File: bms_slave_pcb/bms_slave_pcb.kicad_sch (KiCad schematic)
At the start: 0 parts

Commit message: Add files via upload
Slave Boards Version 1.01 that are ready to be manufactured
Parts:
- added J1: isoSPI Daisy Chain IN, Connector_Molex:Molex_Micro-Fit_3.0_43650-0400_1x04_P3.00mm_Horizontal, symbol Connector:Conn_01x04_Socket
- added J2: isoSPI Daisy Chain OUT, Connector_Molex:Molex_Micro-Fit_3.0_43650-0400_1x04_P3.00mm_Horizontal, symbol Connector:Conn_01x04_Socket
- added U1: LTC6811HGI-1I-3ZZTRPBF, bms_slave_pcb:05-08-1887_ADI, symbol BYU_LIBRARY:LTC6811HG-1-3ZZTRPBF
Connections:
- new net GNDREF: U1.30 (V-), U1.31 (V-)
- new net Power Rail/DRIVE: U1.38 (DRIVE)
- new net Power Rail/VREG: U1.37 (VREG)
- new net Temperature Sensing/GPIO1(MUX_OUT_1): U1.27 (GPIO1)
- new net Temperature Sensing/GPIO2(MUX_OUT_2): U1.28 (GPIO2)
- new net Temperature Sensing/GPIO3: U1.29 (GPIO3)
- new net Temperature Sensing/GPIO4: U1.32 (GPIO4)
- new net Temperature Sensing/GPIO5: U1.33 (GPIO5)
- new net Temperature Sensing/V_REF2: U1.34 (VREF2)
- new net Voltage Taps/C0: U1.26 (C0)
- new net Voltage Taps/C1: U1.24 (C1)
- new net Voltage Taps/C10: U1.6 (C10)
- new net Voltage Taps/C11: U1.4 (C11)
- new net Voltage Taps/C12: U1.2 (C12)
- new net Voltage Taps/C2: U1.22 (C2)
- new net Voltage Taps/C3: U1.20 (C3)
- new net Voltage Taps/C4: U1.18 (C4)
- new net Voltage Taps/C5: U1.16 (C5)
- new net Voltage Taps/C6: U1.14 (C6)
- new net Voltage Taps/C7: U1.12 (C7)
- new net Voltage Taps/C8: U1.10 (C8)
- new net Voltage Taps/C9: U1.8 (C9)
- new net Voltage Taps/S1: U1.25 (S1)
- new net Voltage Taps/S10: U1.7 (S10)
- new net Voltage Taps/S11: U1.5 (S11)
- new net Voltage Taps/S12: U1.3 (S12)
- new net Voltage Taps/S2: U1.23 (S2)
- new net Voltage Taps/S3: U1.21 (S3)
- new net Voltage Taps/S4: U1.19 (S4)
- new net Voltage Taps/S5: U1.17 (S5)
- new net Voltage Taps/S6: U1.15 (S6)
- new net Voltage Taps/S7: U1.13 (S7)
- new net Voltage Taps/S8: U1.11 (S8)
- new net Voltage Taps/S9: U1.9 (S9)
- new net Voltage Taps/VI+: U1.1 (V+)
- new net isoSPI Daisy Chain/+: U1.42 (SCK(IPA))
- new net isoSPI Daisy Chain/-: U1.41 (CSB(IMA))
- new net isoSPI Daisy Chain/DTEN: U1.36 (DTEN)
- new net isoSPI Daisy Chain/I+: U1.48 (IPB)
- new net isoSPI Daisy Chain/I-: U1.47 (IMB)
- new net isoSPI Daisy Chain/IBIAS: U1.45 (IBIAS)
- new net isoSPI Daisy Chain/ICMP: U1.46 (ICMP)
- new net isoSPI Daisy Chain/ISOMD: U1.40 (ISOMD)
- new net isoSPI Daisy Chain/V_REF1: U1.35 (VREF1)
- new net isoSPI Daisy Chain/isoSPIAI+: J1.1 (Pin_1)
- new net isoSPI Daisy Chain/isoSPIAI-: J1.2 (Pin_2)
- new net isoSPI Daisy Chain/isoSPIBI+: J2.1 (Pin_1)
- new net isoSPI Daisy Chain/isoSPIBI-: J2.2 (Pin_2)
- no-connect marks 0 -> 7
Other:
- added sheet FPC Connections (cell_stack.kicad_sch)
- added sheet Power Rail (power_rail.kicad_sch)
- added sheet Temperature Sensing (temp_sensors.kicad_sch)
- added sheet Voltage Taps (voltage_taps.kicad_sch)
- added sheet isoSPI Daisy Chain (isoSPI_daisy_chain.kicad_sch)
- note added: "INPUT"
- note added: "Just as a note for ALL component footprints: I- make ALL caps 0805 handsolder (except voltage tap ones) I- make any resistor dealing with signal logic 0603 handsolder I- make any resistor carrying high current >=0805 I- try to find handsolder footprint versions of any other component"
- note added: "OUTPUT"
- note added: "UnI-used lines for Energy Meter pass thru"
- company: (none) -> BYU Racing
- title: (none) -> BMS Slave 2027
