File: bms_flex_pcb/bms_flex_pcb.kicad_sch (KiCad schematic)
At the start: 0 parts

Commit message: First iteration sent to manufacture
Parts:
- added J1: Flex Connector L, bms_flex_pcb_library:Molex_2190190120_FPC_Board_Connect, symbol Connector:Conn_01x12_Pin
- added J2: Flex Connector R, bms_flex_pcb_library:Molex_2190190120_FPC_Board_Connect, symbol Connector:Conn_01x12_Pin
- added TH1, TH10, TH11, TH12, TH2, TH3, TH4, TH5, TH6, TH7, TH8, TH9: 10k, Resistor_SMD:R_0603_1608Metric_Pad0.98x0.95mm_HandSolder, symbol Device:Thermistor_NTC_US
- added VBUS1, VBUS10, VBUS11, VBUS12, VBUS2, VBUS3, VBUS4, VBUS5, VBUS6, VBUS7, VBUS8, VBUS9, VBUS_GNDREF1: MountingHole_Pad, bms_flex_pcb_library:2026_BMS_Voltage_Tap, symbol Mechanical:MountingHole_Pad
Connections:
- new net: J2.4 (Pin_4), VBUS2.1, VBUS9.1
- new net: J1.1 (Pin_1), VBUS1.1, VBUS6.1
- new net: J1.10 (Pin_10), TH10.1, TH9.1
- new net: J2.10 (Pin_10), TH1.1, TH6.1
- new net: J1.6 (Pin_6), VBUS11.1, VBUS8.1
- new net: J1.3 (Pin_3), TH12.1, TH7.1
- new net: J2.6 (Pin_6), TH11.1, TH8.1
- new net: J1.12 (Pin_12), VBUS10.1, VBUS3.1
- new net: J1.4 (Pin_4), TH2.1, TH5.1
- new net: J1.8 (Pin_8), VBUS4.1
- new net: J2.2 (Pin_2), TH3.1, TH4.1
- new net: J2.12 (Pin_12), VBUS7.1, VBUS_GNDREF1.1
- new net: J2.8 (Pin_8), VBUS12.1, VBUS5.1
- new net GNDREF: J1.11 (Pin_11), J1.2 (Pin_2), J1.5 (Pin_5), J1.7 (Pin_7), J1.9 (Pin_9), J2.1 (Pin_1), J2.11 (Pin_11), J2.3 (Pin_3), J2.5 (Pin_5), J2.7 (Pin_7), J2.9 (Pin_9), TH1.2, TH10.2, TH11.2, TH12.2, TH2.2, TH3.2, TH4.2, TH5.2, TH6.2, TH7.2, TH8.2, TH9.2
Other:
- note added: "GNDREF"
- note added: "MODULE BOTTOM"
- note added: "MODULE TOP"
- note added: "Pin 1 for additional Thermistor?"
- note added: "TH1"
- note added: "TH10"
- note added: "TH11"
- note added: "TH12"
- note added: "TH2"
- note added: "TH3"
- note added: "TH4"
- note added: "TH5"
- note added: "TH6"
- note added: "TH7"
- note added: "TH8"
- note added: "TH9"
- note added: "VBUS1"
- note added: "VBUS10"
- note added: "VBUS11"
- note added: "VBUS12"
- note added: "VBUS2"
- note added: "VBUS3"
- note added: "VBUS4"
- note added: "VBUS5"
- note added: "VBUS6"
- note added: "VBUS7"
- note added: "VBUS8"
- note added: "VBUS9"
