File: bms_slave_pcb_v2/temp_sensors.kicad_sch (KiCad schematic)
At the start: 52 parts, among them IC1 TMUX1308AQPWRQ1, IC2 TMUX1308AQPWRQ1, J3 Extra Thermistor Connector, U2 TLV9002IDR

Commit message: Fixed filenames in BMS Slave PCB V2.01, added equipment wishlist
Other:
- note added: "TH 1-12 are for measuring cell temp TH0, TH13, TH14, & TH15 are ALL EXTRAS"
- note removed: "Nathan TODO: fix/verify the LTC1380 and TMUX1308 footprints Completed 8/2/26"
- note removed: "TH 1I-12 are for measuring cell temp TH0, TH13, TH14, & TH15 are ALL EXTRAS"
- note removed: "if you run out of PCB space on rev 1: then u can ignore & delete this connector"
